File: ec-meter.sch (KiCad schematic (older format))
At the start: 0 parts

Commit message: Added sin wave gen
Parts:
- added 33nF (x3): C, symbol C
- added R? (x3): 22k, symbol R
- added R?: 10k, symbol R
- added U1: LM324, symbol LM324
Connections:
- new net: 33nF.1, R?.1, U1.1
- new net: 33nF.2, R?.2, R?.2, U1.2 (-)
- new net: 33nF.2, R?.1, U1.3 (+)
- new net: 33nF.2, R?.2, U1.6 (-)
- new net: 33nF.1, R?.2, U1.7
- new net +5V: U1.4 (V+)
- new net -5V: U1.11 (V-)
- new net GND: 33nF.1, R?.1, R?.1, U1.5 (+)
Changed lines of the file:
@@
 LIBS:valves
 LIBS:visgence_parts
+LIBS:ec-meter-cache
 EELAYER 25 0
 EELAYER END
@@
 Comment4 ""
 $EndDescr
+$Comp
+L LM324 U1
+U 1 1 58825C06
+P 2100 1850
+F 0 "U1" H 2100 2050 50  0000 L CNN
+F 1 "LM324" H 2100 1650 50  0000 L CNN
+F 2 "" H 2050 1950 50  0000 C CNN
+F 3 "" H 2150 2050 50  0000 C CNN
+	1    2100 1850
+	1    0    0    -1
+$EndComp
+$Comp
+L LM324 U1
+U 2 1 58825C58
+P 3550 1850
+F 0 "U1" H 3550 2050 50  0000 L CNN
+F 1 "LM324" H 3550 1650 50  0000 L CNN
+F 2 "" H 3500 1950 50  0000 C CNN
+F 3 "" H 3600 2050 50  0000 C CNN
+	2    3550 1850
+	1    0    0    -1
+$EndComp
+$Comp
+L GND #PWR?
+U 1 1 58825CF9
+P 3100 2150
+F 0 "#PWR?" H 3100 1900 50  0001 C CNN
+F 1 "GND" H 3100 2000 50  0000 C CNN
+F 2 "" H 3100 2150 50  0000 C CNN
+F 3 "" H 3100 2150 50  0000 C CNN
+	1    3100 2150
+	1    0    0    -1
+$EndComp
+Wire Wire Line
+	3100 1750 3100 2150
+Wire Wire Line
+	3100 1750 3250 1750
+$Comp
+L R R?
+U 1 1 58825D49
+P 2800 1950
+F 0 "R?" V 2880 1950 50  0000 C CNN
+F 1 "22k" V 2800 1950 50  0000 C CNN
+F 2 "" V 2730 1950 50  0000 C CNN
+F 3 "" H 2800 1950 50  0000 C CNN
+	1    2800 1950
+	0    -1   -1   0
+$EndComp
+Wire Wire Line
+	2400 1850 2400 2400
+Wire Wire Line
+	2400 1950 2650 1950
+Wire Wire Line
+	2950 1950 3250 1950
+$Comp
+L R R?
+U 1 1 58825E0B
+P 1600 2200
+F 0 "R?" V 1680 2200 50  0000 C CNN
+F 1 "22k" V 1600 2200 50  0000 C CNN
+F 2 "" V 1530 2200 50  0000 C CNN
+F 3 "" H 1600 2200 50  0000 C CNN
+	1    1600 2200
+	-1   0    0    1
+$EndComp
+Wire Wire Line
+	1600 2050 1600 1950
+Wire Wire Line
+	1350 1950 1800 1950
+$Comp
+L GND #PWR?
+U 1 1 58825E8A
+P 1600 2450
+F 0 "#PWR?" H 1600 2200 50  0001 C CNN
+F 1 "GND" H 1600 2300 50  0000 C CNN
+F 2 "" H 1600 2450 50  0000 C CNN
+F 3 "" H 1600 2450 50  0000 C CNN
+	1    1600 2450
+	1    0    0    -1
+$EndComp
+$Comp
+L R R?
+U 1 1 58825EA1
+P 1350 2200
+F 0 "R?" V 1430 2200 50  0000 C CNN
+F 1 "10k" V 1350 2200 50  0000 C CNN
+F 2 "" V 1280 2200 50  0000 C CNN
+F 3 "" H 1350 2200 50  0000 C CNN
+	1    1350 2200
+	-1   0    0    1
+$EndComp
+Wire Wire Line
+	1350 1950 1350 2050
+Connection ~ 1600 1950
+Wire Wire Line
+	1350 2350 1350 2400
+Wire Wire Line
+	1350 2400 1600 2400
+Wire Wire Line
+	1600 2350 1600 2450
+Connection ~ 1600 2400
+$Comp
+L C 33nF
+U 1 1 58825F83
+P 2000 2400
+F 0 "33nF" H 2025 2500 50  0000 L CNN
+F 1 "C" H 2025 2300 50  0000 L CNN
+F 2 "" H 2038 2250 50  0000 C CNN
+F 3 "" H 2000 2400 50  0000 C CNN
+	1    2000 2400
+	0    1    1    0
+$EndComp
+Wire Wire Line
+	2400 2400 2150 2400
+Connection ~ 2400 1950
+Wire Wire Line
+	1850 2400 1750 2400
+Wire Wire Line
+	1750 2400 1750 1950
+Connection ~ 1750 1950
+$Comp
+L C 33nF
+U 1 1 5882608A
+P 1050 1900
+F 0 "33nF" H 1075 2000 50  0000 L CNN
+F 1 "C" H 1075 1800 50  0000 L CNN
+F 2 "" H 1088 1750 50  0000 C CNN
+F 3 "" H 1050 1900 50  0000 C CNN
+	1    1050 1900
+	-1   0    0    1
+$EndComp
+$Comp
+L GND #PWR?
+U 1 1 588260EB
+P 1050 2200
+F 0 "#PWR?" H 1050 1950 50  0001 C CNN
+F 1 "GND" H 1050 2050 50  0000 C CNN
+F 2 "" H 1050 2200 50  0000 C CNN
+F 3 "" H 1050 2200 50  0000 C CNN
+	1    1050 2200
+	1    0    0    -1
+$EndComp
+Wire Wire Line
+	1050 1750 1800 1750
+Wire Wire Line
+	1050 2050 1050 2200
+$Comp
+L R R?
+U 1 1 5882614B
+P 2800 1250
+F 0 "R?" V 2880 1250 50  0000 C CNN
+F 1 "22k" V 2800 1250 50  0000 C CNN
+F 2 "" V 2730 1250 50  0000 C CNN
+F 3 "" H 2800 1250 50  0000 C CNN
+	1    2800 1250
+	0    -1   -1   0
+$EndComp
+Wire Wire Line
+	1750 1250 2650 1250
+Wire Wire Line
+	1750 1250 1750 1750
+Connection ~ 1750 1750
+Wire Wire Line
+	3850 1850 4000 1850
+Wire Wire Line
+	4000 2400 4000 1250
+$Comp
+L C 33nF
+U 1 1 58826293
+P 3500 2400
+F 0 "33nF" H 3525 2500 50  0000 L CNN
+F 1 "C" H 3525 2300 50  0000 L CNN
+F 2 "" H 3538 2250 50  0000 C CNN
+F 3 "" H 3500 2400 50  0000 C CNN
+	1    3500 2400
+	0    1    1    0
+$EndComp
+Wire Wire Line
+	3650 2400 4000 2400
+Connection ~ 4000 1850
+Wire Wire Line
+	3350 2400 3200 2400
+Wire Wire Line
+	3200 2400 3200 1950
+Connection ~ 3200 1950
+$Comp
+L +5V #PWR?
+U 1 1 5882641D
+P 2000 1450
+F 0 "#PWR?" H 2000 1300 50  0001 C CNN
+F 1 "+5V" H 2000 1590 50  0000 C CNN
+F 2 "" H 2000 1450 50  0000 C CNN
+F 3 "" H 2000 1450 50  0000 C CNN
+	1    2000 1450
+	1    0    0    -1
+$EndComp
+Wire Wire Line
+	2000 1550 2000 1450
+$Comp
+L -5V #PWR?
+U 1 1 588265C4
+P 2150 2200
+F 0 "#PWR?" H 2150 2300 50  0001 C CNN
+F 1 "-5V" H 2150 2350 50  0000 C CNN
+F 2 "" H 2150 2200 50  0000 C CNN
+F 3 "" H 2150 2200 50  0000 C CNN
+	1    2150 2200
+	-1   0    0    1
+$EndComp
+Wire Wire Line
+	2150 2200 2000 2200
+Wire Wire Line
+	2000 2200 2000 2150
+Wire Wire Line
+	4000 1250 2950 1250
 $EndSCHEMATC
